File: circuit/robot_mini_r1.sch (EAGLE design)
At the start: 10 parts, among them M1 SERVO-FLIPPED, M2 SERVO-1, M3 SERVO-1, U1 ESP01

Commit message: web stuff works, more settings, PCB configurable
Parts:
- removed SJ1: SOLDERJUMPERNO, robot:SOLDERJUMPERNO
- added LED1: (no value), robot:LED5MM
- added R1: 220Ω, robot:RESISTORAXIAL-0.3-NOVAL
- U$9: value TEXT-INFO-MINI -> TEXT-INFO-INVISIBLE; device robot:TEXT-INFO-MINI -> robot:TEXT-INFO-INVISIBLE
Connections:
- removed net N$1: SJ1.2, U1.TXD
- new net N$9: LED1.A, R1.2
- new net SERVO-AUX: M3.SIG, U1.RXD
- net 3.3V: now also R1.1; no longer U1.CH_PD
- net GND: now also LED1.C
- net SERVO-LEFT: no longer M3.SIG, SJ1.1
- net SERVO-RIGHT: now also U1.GPIO0; no longer U1.GPIO0(P)
Other:
- moved on the sheet: U1
