File: circuit/dirtcheaprx.sch (EAGLE design)
At the start: 11 parts, among them M1 SERVO-FLIPPED, M2 SERVO-1, M3 SERVO-1, U1 ESP01

Commit message: PCBs, first proto batch
Parts:
- removed BATTERY: (no value), robot:BATTERY-WIRE-CONN
- removed M1: SERVO-FLIPPED, robot:SERVO-FLIPPED
- removed M2, M3: SERVO-1, robot:SERVO-1
- removed U$9: TEXT-INFO-INVISIBLE, robot:TEXT-INFO-INVISIBLE
- added BAT1: (no value), dirtcheaprx:BATTERY-WIRE-CONN
- added R2: 1KΩ, dirtcheaprx:RESISTOR0603-RES
- added R3: 470Ω, dirtcheaprx:RESISTOR0603-RES
- added SERVO1, SERVO2, SERVO3: SERVO-1, dirtcheaprx:SERVO-1
- added SJ1, SJ2, SJ3: SOLDERJUMPERNO, dirtcheaprx:SOLDERJUMPERNO
- added TP1, TP2, TP3, TP4, TP5: TPPAD1-13, dirtcheaprx:TPPAD1-13
- C1: value (none) -> 100uF; device robot:CAP_POLPTH1 -> dirtcheaprx:CAP0603-CAP
- C2: value (none) -> 1u; device robot:CAPPTH -> dirtcheaprx:CAP0603-CAP
- IC1: value (none) -> MCP1700; device robot:V_REG_78XXTO-92 -> dirtcheaprx:V_REG_78XX-SOT
- LED1: device robot:LED5MM -> dirtcheaprx:LED5MM
- R1: value 220Ω -> 7K5Ω; device robot:RESISTORAXIAL-0.3-NOVAL -> dirtcheaprx:RESISTOR0603-RES
- U1: value ESP01 -> (none); device robot:ESP01 -> dirtcheaprx:ESP12SMD
Connections:
- removed net SERVO-AUX: M3.SIG, U1.RXD
- removed net SERVO-LEFT: M1.SIG, U1.GPIO2
- removed net SERVO-RIGHT: M2.SIG, U1.GPIO0
- new net ADC: R1.1, R2.2, U1.ADC
- new net LED: R3.1, U1.GPIO4
- new net N$1: LED1.A, R3.2
- new net N$10: TP3.TP, U1.RX
- new net N$11: TP4.TP, U1.GPIO0
- new net N$2: SERVO1.PWR, SJ1.1
- new net N$3: SERVO2.PWR, SJ2.1
- new net N$4: SERVO3.PWR, SJ3.1
- new net N$8: TP1.TP, U1.RESET
- new net SIG-L: SERVO3.SIG, U1.GPIO13
- new net SIG-RIGHT: SERVO1.SIG, U1.GPIO15
- new net SIG-WEAP: SERVO2.SIG, U1.GPIO5
- net +6V: now also BAT1.+, C2.1, R1.2, SJ1.2, SJ2.2, SJ3.2; no longer BATTERY.+, C1.+, M1.PWR, M2.PWR, M3.PWR
- net 3.3V: now also C1.1, TP5.TP, U1.CH_PD; no longer C2.1, R1.1
- net GND: now also BAT1.-, C1.2, R2.1, SERVO1.GND, SERVO2.GND, SERVO3.GND; no longer BATTERY.-, C1.-, M1.GND, M2.GND, M3.GND
- net N$9: now also TP2.TP, U1.TX; no longer LED1.A, R1.2
Other:
- note added: "8.5V in to 1.0V out"
- moved on the sheet: C2, IC1, LED1, R1
