File: circuit/programmer.brd (EAGLE design)
At the start: 100 x 100 mm, 5 parts, among them U1 TEENSY_3.0_DIL, X1 ESP01, X2 DIRTCHEAPRX-PROG-MINI, X3 DIRTCHEAPRX-PROG-NANO

Commit message: progress on programmer pcb
Parts:
- added D1: (no value), dirtcheaprx:SOD-323
- added LED1, LED2, LED3, LED4, LED5: (no value), dirtcheaprx:LED5MM
- added R1, R2, R3, R4, R5: (no value), dirtcheaprx:0603-RES
- added S2: (no value), dirtcheaprx:TACTILE-PTH
Connections:
- new net LED-BAD: R2.1, U1.6
- new net LED-DATA-DOWN: R4.1, U1.4
- new net LED-DATA-UP: R3.1, U1.5
- new net LED-GOOD: R1.1, U1.7
- new net LED-V: R5.1, U1.3
- new net N$1: D1.1, U1.11
- new net N$2: LED1.A, R1.2
- new net N$4: LED3.A, R3.2
- new net N$5: LED4.A, R4.2
- new net N$6: LED5.A, R5.2
- net BTN: now also U1.2
- net GND: now also LED1.K, LED2.K, LED3.K, LED4.K, LED5.K, S2.3, S2.4
- net N$3: now also LED2.A, R2.2; no longer U1.3
- net RST: now also D1.2, S2.1, S2.2; no longer U1.11
Routing:
- net LED-GOOD: track 0.00 -> 40.1 mm
- net LED-BAD: track 0.00 -> 38.2 mm
- net LED-DATA-UP: track 0.00 -> 36.4 mm
- net LED-DATA-DOWN: track 0.00 -> 34.5 mm
- net BTN: track 0.00 -> 34.2 mm
- net LED-V: track 0.00 -> 32.7 mm
- net RST: track 161.0 -> 182.1 mm
- net N$1: track 0.00 -> 3.26 mm
- net N$6: track 0.00 -> 2.88 mm
- net N$5: track 0.00 -> 2.88 mm
- net N$4: track 0.00 -> 2.88 mm
- net N$3: track 0.00 -> 2.88 mm
- net N$2: track 0.00 -> 2.88 mm
- net TX: track 199.7 -> 198.8 mm
- net RX: track 171.8 -> 171.1 mm
Other:
- board text added: "+3V3 Status"
- board text added: "Data"
- board text added: "ERROR"
- board text added: "Go!!!"
- board text added: "Good!!!"
- board text added: "Reset"
Changed lines of the file:
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@@
 <hole x="96" y="96" drill="3"/>
 <hole x="4" y="96" drill="3"/>
+<text x="77" y="4" size="1.778" layer="21" ratio="10">Go!!!</text>
+<text x="89" y="14" size="1.778" layer="21" font="vector" ratio="10" rot="R180" align="center-left">+3V3 Status</text>
+<text x="86" y="21" size="1.778" layer="21" font="vector" ratio="10" rot="R180" align="center-left">Data</text>
+<text x="86" y="28" size="1.778" layer="21" font="vector" ratio="10" rot="R180" align="center-left">Data</text>
+<text x="89" y="42" size="1.778" layer="21" font="vector" ratio="10" rot="R180" align="center-left">Good!!!</text>
+<text x="89" y="35" size="1.778" layer="21" font="vector" ratio="10" rot="R180" align="center-left">ERROR</text>
+<wire x1="88" y1="27" x2="88" y2="30" width="0.4064" layer="21"/>
+<wire x1="88" y1="30" x2="87" y2="29" width="0.4064" layer="21"/>
+<wire x1="87" y1="29" x2="89" y2="29" width="0.4064" layer="21"/>
+<wire x1="89" y1="29" x2="88" y2="30" width="0.4064" layer="21"/>
+<wire x1="88" y1="22" x2="88" y2="19" width="0.4064" layer="21"/>
+<wire x1="88" y1="19" x2="87" y2="20" width="0.4064" layer="21"/>
+<wire x1="87" y1="20" x2="89" y2="20" width="0.4064" layer="21"/>
+<wire x1="89" y1="20" x2="88" y2="19" width="0.4064" layer="21"/>
+<text x="88" y="52" size="1.778" layer="21" font="vector" ratio="10" rot="R180" align="center-left">Reset</text>
 </plain>
 <attributes>
@@
 <element name="S1" library="dirtcheaprx" package="TACTILE-PTH" value="" x="87" y="5"/>
 <element name="U1" library="dirtcheaprx" package="TEENSY_3.0-3.2&amp;LC_DIL" value="TEENSY_3.0_DIL" x="50" y="20" rot="R180"/>
+<element name="D1" library="dirtcheaprx" package="SOD-323" value="" x="62" y="34"/>
+<element name="S2" library="dirtcheaprx" package="TACTILE-PTH" value="" x="93" y="52" rot="R180"/>
+<element name="LED1" library="dirtcheaprx" package="LED5MM" value="" x="96" y="42"/>
+<element name="LED2" library="dirtcheaprx" package="LED5MM" value="" x="96" y="35"/>
+<element name="LED3" library="dirtcheaprx" package="LED5MM" value="" x="96" y="28"/>
+<element name="LED4" library="dirtcheaprx" package="LED5MM" value="" x="96" y="21"/>
+<element name="LED5" library="dirtcheaprx" package="LED5MM" value="" x="96" y="14"/>
+<element name="R1" library="dirtcheaprx" package="0603-RES" value="" x="91" y="42"/>
+<element name="R2" library="dirtcheaprx" package="0603-RES" value="" x="91" y="35"/>
+<element name="R3" library="dirtcheaprx" package="0603-RES" value="" x="91" y="28"/>
+<element name="R4" library="dirtcheaprx" package="0603-RES" value="" x="91" y="21"/>
+<element name="R5" library="dirtcheaprx" package="0603-RES" value="" x="91" y="14"/>
 </elements>
 <signals>
@@
 <contactref element="X3" pad="TX"/>
 <contactref element="U1" pad="0"/>
-<wire x1="57.62" y1="6.03" x2="53" y2="6.03" width="0.2032" layer="1"/>
-<wire x1="53" y1="6.03" x2="53" y2="59" width="0.2032" layer="1"/>
+<wire x1="57.62" y1="6.03" x2="54.393159375" y2="6.03" width="0.2032" layer="1"/>
+<wire x1="54.393159375" y1="6.03" x2="53" y2="7.423159375" width="0.2032" layer="1"/>
+<wire x1="53" y1="7.423159375" x2="53" y2="59" width="0.2032" layer="1"/>
 <wire x1="6.175" y1="73.8225" x2="4" y2="75.9975" width="0.2032" layer="1"/>
 <wire x1="4" y1="75.9975" x2="4" y2="79" width="0.2032" layer="1"/>
@@
 <wire x1="37.7" y1="85.7" x2="36.3" y2="85.7" width="0.2032" layer="16"/>
 <wire x1="36.3" y1="85.7" x2="34.6" y2="84" width="0.2032" layer="16"/>
-<contactref element="U1" pad="11"/>
 <wire x1="73.1" y1="86.6" x2="69.7" y2="90" width="0.2032" layer="16"/>
 <wire x1="69.7" y1="90" x2="68.5" y2="90" width="0.2032" layer="16"/>
@@
 <wire x1="44" y1="94" x2="43" y2="93" width="0.2032" layer="16"/>
 <wire x1="43" y1="93" x2="41" y2="93" width="0.2032" layer="16"/>
-<wire x1="57.62" y1="33.97" x2="78" y2="54.35" width="0.2032" layer="1"/>
-<wire x1="78" y1="54.35" x2="78" y2="73" width="0.2032" layer="1"/>
 <wire x1="78" y1="73" x2="73.1" y2="77.9" width="0.2032" layer="1"/>
 <wire x1="73.1" y1="77.9" x2="73.1" y2="86.6" width="0.2032" layer="1"/>
@@
 <wire x1="67.5" y1="91" x2="66" y2="91" width="0.2032" layer="16"/>
 <wire x1="66" y1="91" x2="63" y2="94" width="0.2032" layer="16"/>
+<contactref element="D1" pad="2"/>
+<wire x1="63.15" y1="34" x2="72" y2="34" width="0.2032" layer="1"/>
+<wire x1="72" y1="34" x2="78" y2="40" width="0.2032" layer="1"/>
+<wire x1="78" y1="40" x2="78" y2="49" width="0.2032" layer="1"/>
+<contactref element="S2" pad="1"/>
+<contactref element="S2" pad="2"/>
+<wire x1="78" y1="49.7394" x2="78" y2="73" width="0.2032" layer="1"/>
+<wire x1="96.2512" y1="49.7394" x2="89.7488" y2="49.7394" width="0.2032" layer="1"/>
+<wire x1="89.7488" y1="49.7394" x2="78" y2="49.7394" width="0.2032" layer="1"/>
+<wire x1="78" y1="49.7394" x2="78" y2="49" width="0.2032" layer="1"/>
 </signal>
 <signal name="RX">
@@
 <contactref element="X3" pad="RX"/>
 <contactref element="U1" pad="1"/>
-<wire x1="57.62" y1="8.57" x2="54" y2="8.57" width="0.2032" layer="1"/>
-<wire x1="54" y1="8.57" x2="54" y2="58" width="0.2032" layer="1"/>
+<wire x1="57.62" y1="8.57" x2="55.088528125" y2="8.57" width="0.2032" layer="1"/>
+<wire x1="55.088528125" y1="8.57" x2="54" y2="9.658528125" width="0.2032" layer="1"/>
+<wire x1="54" y1="9.658528125" x2="54" y2="58" width="0.2032" layer="1"/>
 <wire x1="13.795" y1="76.3625" x2="17.6375" y2="76.3625" width="0.2032" layer="1"/>
 <wire x1="17.6375" y1="76.3625" x2="21" y2="73" width="0.2032" layer="1"/>
@@
 <via x="67" y="92" extent="1-16" drill="0.3" shape="octagon"/>
 <via x="84" y="79" extent="1-16" drill="0.3" shape="octagon"/>
+<contactref element="S2" pad="3"/>
+<contactref element="S2" pad="4"/>
+<contactref element="LED1" pad="K"/>
+<contactref element="LED5" pad="K"/>
+<contactref element="LED4" pad="K"/>
+<contactref element="LED3" pad="K"/>
+<contactref element="LED2" pad="K"/>
 </signal>
 <signal name="A0">
@@
 <wire x1="28" y1="94" x2="28" y2="87.4" width="0.8128" layer="16"/>
 </signal>
-<signal name="N$3">
-<contactref element="U1" pad="3"/>
-</signal>
 <signal name="BTN">
 <contactref element="S1" pad="1"/>
 <contactref element="S1" pad="2"/>
-<wire x1="83.7488" y1="7.2606" x2="90.2512" y2="7.2606" width="0" layer="19" extent="1-1"/>
+<contactref element="U1" pad="2"/>
+<wire x1="90.2512" y1="7.2606" x2="83.7488" y2="7.2606" width="0.2032" layer="1"/>
+<wire x1="83.7488" y1="7.2606" x2="76.7394" y2="7.2606" width="0.2032" layer="1"/>
+<wire x1="76.7394" y1="7.2606" x2="72.89" y2="11.11" width="0.2032" layer="1"/>
+<wire x1="72.89" y1="11.11" x2="57.62" y2="11.11" width="0.2032" layer="1"/>
+</signal>
+<signal name="N$1">
+<contactref element="U1" pad="11"/>
+<contactref element="D1" pad="1"/>
+<wire x1="57.62" y1="33.97" x2="60.85" y2="33.97" width="0.2032" layer="1"/>
+<wire x1="60.85" y1="33.97" x2="60.85" y2="34" width="0.2032" layer="1"/>
+</signal>
+<signal name="N$2">
+<contactref element="LED1" pad="A"/>
+<contactref element="R1" pad="2"/>
+<wire x1="91.85" y1="42" x2="94.73" y2="42" width="0.2032" layer="1"/>
+</signal>
+<signal name="N$3">
+<contactref element="LED2" pad="A"/>
+<contactref element="R2" pad="2"/>
+<wire x1="91.85" y1="35" x2="94.73" y2="35" width="0.2032" layer="1"/>
+</signal>
+<signal name="N$4">
+<contactref element="LED3" pad="A"/>
+<contactref element="R3" pad="2"/>
+<wire x1="91.85" y1="28" x2="94.73" y2="28" width="0.2032" layer="1"/>
+</signal>
+<signal name="N$5">
+<contactref element="LED4" pad="A"/>
+<contactref element="R4" pad="2"/>
+<wire x1="91.85" y1="21" x2="94.73" y2="21" width="0.2032" layer="1"/>
+</signal>
+<signal name="N$6">
+<contactref element="LED5" pad="A"/>
+<contactref element="R5" pad="2"/>
+<wire x1="91.85" y1="14" x2="94.73" y2="14" width="0.2032" layer="1"/>
+</signal>
+<signal name="LED-GOOD">
+<contactref element="R1" pad="1"/>
+<contactref element="U1" pad="7"/>
+<wire x1="57.62" y1="23.81" x2="66.81" y2="23.81" width="0.2032" layer="1"/>
+<wire x1="66.81" y1="23.81" x2="85" y2="42" width="0.2032" layer="1"/>
+<wire x1="85" y1="42" x2="90.15" y2="42" width="0.2032" layer="1"/>
+</signal>
+<signal name="LED-BAD">
+<contactref element="R2" pad="1"/>
+<contactref element="U1" pad="6"/>
+<wire x1="57.62" y1="21.27" x2="68.27" y2="21.27" width="0.2032" layer="1"/>
+<wire x1="68.27" y1="21.27" x2="82" y2="35" width="0.2032" layer="1"/>
+<wire x1="82" y1="35" x2="90.15" y2="35" width="0.2032" layer="1"/>
+</signal>
+<signal name="LED-DATA-UP">
+<contactref element="R3" pad="1"/>
+<contactref element="U1" pad="5"/>
+<wire x1="57.62" y1="18.73" x2="70.73" y2="18.73" width="0.2032" layer="1"/>
+<wire x1="70.73" y1="18.73" x2="80" y2="28" width="0.2032" layer="1"/>
+<wire x1="80" y1="28" x2="90.15" y2="28" width="0.2032" layer="1"/>
+</signal>
+<signal name="LED-DATA-DOWN">
+<contactref element="R4" pad="1"/>
+<contactref element="U1" pad="4"/>
+<wire x1="57.62" y1="16.19" x2="73.19" y2="16.19" width="0.2032" layer="1"/>
+<wire x1="73.19" y1="16.19" x2="78" y2="21" width="0.2032" layer="1"/>
+<wire x1="78" y1="21" x2="90.15" y2="21" width="0.2032" layer="1"/>
+</signal>
+<signal name="LED-V">
+<contactref element="R5" pad="1"/>
+<contactref element="U1" pad="3"/>
+<wire x1="57.62" y1="13.65" x2="87.65" y2="13.65" width="0.2032" layer="1"/>
+<wire x1="87.65" y1="13.65" x2="88" y2="14" width="0.2032" layer="1"/>
+<wire x1="88" y1="14" x2="90.15" y2="14" width="0.2032" layer="1"/>
 </signal>
 </signals>

Commit message: work on programmer pcb
Parts:
- added C1: (no value), dirtcheaprx:CPOL-RADIAL-100UF-25V
- added C2: (no value), dirtcheaprx:CAP-PTH-SMALL2
- added D2: (no value), dirtcheaprx:SOD-323
- added IC1: (no value), dirtcheaprx:SOT223
- added S3: (no value), dirtcheaprx:TACTILE-PTH
- added X4: ESP01, dirtcheaprx:ESP01
- moved S2 85.0 mm to (8.00, 54.0), turned to 0 degrees
- moved X1 10.0 mm to (10.0, 72.0)
- moved X2 10.0 mm to (68.0, 56.0)
- moved X3 10.0 mm to (52.0, 56.0)
Connections:
- new net 3.3V: U1.3.3V
- new net N$7: D2.1, U1.12
- new net RX2: U1.10, X4.RX
- new net SCANNER-RST: U1.8, X4.RST
- new net TX2: U1.9, X4.TX
- net +3V3: now also C2.1, IC1.2, IC1.4, X4.CH_PD, X4.GPIO0, X4.VCC; no longer U1.3.3V
- net BOOT: now also D2.2, S3.1, S3.2; no longer U1.12
- net GND: now also C1.2, C2.2, IC1.1, S3.3, S3.4, X4.GND
- net VIN: now also C1.1, IC1.3
Routing:
- net TX2: track 0.00 -> 62.7 mm, vias 0 -> 2
- net RX2: track 0.00 -> 60.0 mm, vias 0 -> 2
- net SCANNER-RST: track 0.00 -> 53.4 mm, vias 0 -> 2
- net BOOT: track 136.0 -> 162.4 mm, vias 1 -> 3
- net RST: track 182.1 -> 167.9 mm
- net RX: track 171.1 -> 160.7 mm
- net A0: track 98.5 -> 88.5 mm
- net TX: track 198.8 -> 189.8 mm
- net N$7: track 0.00 -> 3.24 mm
- net VIN: track 161.1 -> 159.4 mm
- net +3V3: track 100.7 -> 101.8 mm, vias 0 -> 2
Other:
- board size 100 x 100 mm -> 100 x 90 mm
- board text added: "Boot"
- board text added: "Good"
- board text added: "Scanner"
- board text removed: "Good!!!"
