File: circuit/programmer.sch (EAGLE design)
At the start: 5 parts, among them U1 TEENSY_3.0_DIL, X1 ESP01, X2 DIRTCHEAPRX-PROG-MINI, X3 DIRTCHEAPRX-PROG-NANO

Commit message: progress on programmer pcb
Parts:
- added D1: (no value), dirtcheaprx:DIODESOD
- added LED1, LED2, LED3, LED4, LED5: (no value), dirtcheaprx:LED5MM
- added R1, R2, R3, R4, R5: (no value), dirtcheaprx:RESISTOR0603-RES
- added S2: (no value), dirtcheaprx:TAC_SWITCHPTH
Connections:
- new net LED-BAD: R2.1, U1.6/PWM
- new net LED-DATA-DOWN: R4.1, U1.4/PWM
- new net LED-DATA-UP: R3.1, U1.5/PWM
- new net LED-GOOD: R1.1, U1.7/RX3
- new net LED-V: R5.1, U1.3/PWM
- new net N$1: D1.C, U1.11/MOSI
- new net N$2: LED1.A, R1.2
- new net N$4: LED3.A, R3.2
- new net N$5: LED4.A, R4.2
- new net N$6: LED5.A, R5.2
- net BTN: now also U1.2
- net GND: now also LED1.C, LED2.C, LED3.C, LED4.C, LED5.C, S2.3, S2.4
- net N$3: now also LED2.A, R2.2; no longer U1.3/PWM
- net RST: now also D1.A, S2.1, S2.2; no longer U1.11/MOSI
Changed lines of the file:
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@@
 <part name="GND4" library="dirtcheaprx" deviceset="GND" device=""/>
 <part name="GND5" library="dirtcheaprx" deviceset="GND" device=""/>
+<part name="D1" library="dirtcheaprx" deviceset="DIODE" device="SOD"/>
+<part name="S2" library="dirtcheaprx" deviceset="TAC_SWITCH" device="PTH"/>
+<part name="GND6" library="dirtcheaprx" deviceset="GND" device=""/>
+<part name="LED1" library="dirtcheaprx" deviceset="LED" device="5MM"/>
+<part name="LED2" library="dirtcheaprx" deviceset="LED" device="5MM"/>
+<part name="LED3" library="dirtcheaprx" deviceset="LED" device="5MM"/>
+<part name="LED4" library="dirtcheaprx" deviceset="LED" device="5MM"/>
+<part name="LED5" library="dirtcheaprx" deviceset="LED" device="5MM"/>
+<part name="R1" library="dirtcheaprx" deviceset="RESISTOR" device="0603-RES"/>
+<part name="R2" library="dirtcheaprx" deviceset="RESISTOR" device="0603-RES"/>
+<part name="R3" library="dirtcheaprx" deviceset="RESISTOR" device="0603-RES"/>
+<part name="R4" library="dirtcheaprx" deviceset="RESISTOR" device="0603-RES"/>
+<part name="R5" library="dirtcheaprx" deviceset="RESISTOR" device="0603-RES"/>
+<part name="GND7" library="dirtcheaprx" deviceset="GND" device=""/>
 </parts>
 <sheets>
@@
 <instance part="GND4" gate="1" x="154.94" y="12.7"/>
 <instance part="GND5" gate="1" x="190.5" y="-10.16"/>
+<instance part="D1" gate="G$1" x="91.44" y="12.7"/>
+<instance part="S2" gate="S" x="182.88" y="-25.4"/>
+<instance part="GND6" gate="1" x="190.5" y="-33.02"/>
+<instance part="LED1" gate="G$1" x="246.38" y="22.86" rot="R90"/>
+<instance part="LED2" gate="G$1" x="246.38" y="12.7" rot="R90"/>
+<instance part="LED3" gate="G$1" x="246.38" y="2.54" rot="R90"/>
+<instance part="LED4" gate="G$1" x="246.38" y="-7.62" rot="R90"/>
+<instance part="LED5" gate="G$1" x="246.38" y="-17.78" rot="R90"/>
+<instance part="R1" gate="G$1" x="238.76" y="22.86"/>
+<instance part="R2" gate="G$1" x="238.76" y="12.7"/>
+<instance part="R3" gate="G$1" x="238.76" y="2.54"/>
+<instance part="R4" gate="G$1" x="238.76" y="-7.62"/>
+<instance part="R5" gate="G$1" x="238.76" y="-17.78"/>
+<instance part="GND7" gate="1" x="254" y="-25.4"/>
 </instances>
 <busses>
@@
 </segment>
 <segment>
-<pinref part="U1" gate="G$1" pin="11/MOSI"/>
-<wire x1="106.68" y1="12.7" x2="101.6" y2="12.7" width="0.1524" layer="91"/>
-<label x="101.6" y="12.7" size="1.27" layer="95" rot="R180" xref="yes"/>
+<pinref part="D1" gate="G$1" pin="A"/>
+<wire x1="88.9" y1="12.7" x2="83.82" y2="12.7" width="0.1524" layer="91"/>
+<label x="83.82" y="12.7" size="1.27" layer="95" rot="R180" xref="yes"/>
+</segment>
+<segment>
+<pinref part="S2" gate="S" pin="1"/>
+<wire x1="177.8" y1="-25.4" x2="175.26" y2="-25.4" width="0.1524" layer="91"/>
+<pinref part="S2" gate="S" pin="2"/>
+<wire x1="175.26" y1="-25.4" x2="170.18" y2="-25.4" width="0.1524" layer="91"/>
+<wire x1="177.8" y1="-27.94" x2="175.26" y2="-27.94" width="0.1524" layer="91"/>
+<wire x1="175.26" y1="-27.94" x2="175.26" y2="-25.4" width="0.1524" layer="91"/>
+<label x="170.18" y="-25.4" size="1.27" layer="95" rot="R180" xref="yes"/>
 </segment>
 </net>
@@
 <wire x1="187.96" y1="-5.08" x2="190.5" y2="-5.08" width="0.1524" layer="91"/>
 </segment>
+<segment>
+<pinref part="S2" gate="S" pin="3"/>
+<pinref part="GND6" gate="1" pin="GND"/>
+<wire x1="187.96" y1="-25.4" x2="190.5" y2="-25.4" width="0.1524" layer="91"/>
+<wire x1="190.5" y1="-25.4" x2="190.5" y2="-27.94" width="0.1524" layer="91"/>
+<pinref part="S2" gate="S" pin="4"/>
+<wire x1="190.5" y1="-27.94" x2="190.5" y2="-30.48" width="0.1524" layer="91"/>
+<wire x1="187.96" y1="-27.94" x2="190.5" y2="-27.94" width="0.1524" layer="91"/>
+</segment>
+<segment>
+<pinref part="LED1" gate="G$1" pin="C"/>
+<pinref part="GND7" gate="1" pin="GND"/>
+<wire x1="251.46" y1="22.86" x2="254" y2="22.86" width="0.1524" layer="91"/>
+<wire x1="254" y1="22.86" x2="254" y2="12.7" width="0.1524" layer="91"/>
+<pinref part="LED5" gate="G$1" pin="C"/>
+<wire x1="254" y1="12.7" x2="254" y2="2.54" width="0.1524" layer="91"/>
+<wire x1="254" y1="2.54" x2="254" y2="-7.62" width="0.1524" layer="91"/>
+<wire x1="254" y1="-7.62" x2="254" y2="-17.78" width="0.1524" layer="91"/>
+<wire x1="254" y1="-17.78" x2="254" y2="-22.86" width="0.1524" layer="91"/>
+<wire x1="251.46" y1="-17.78" x2="254" y2="-17.78" width="0.1524" layer="91"/>
+<pinref part="LED4" gate="G$1" pin="C"/>
+<wire x1="251.46" y1="-7.62" x2="254" y2="-7.62" width="0.1524" layer="91"/>
+<pinref part="LED3" gate="G$1" pin="C"/>
+<wire x1="251.46" y1="2.54" x2="254" y2="2.54" width="0.1524" layer="91"/>
+<pinref part="LED2" gate="G$1" pin="C"/>
+<wire x1="251.46" y1="12.7" x2="254" y2="12.7" width="0.1524" layer="91"/>
+</segment>
 </net>
 <net name="A0" class="0">
@@
 <wire x1="152.4" y1="40.64" x2="157.48" y2="40.64" width="0.1524" layer="91"/>
 <label x="157.48" y="40.64" size="1.27" layer="95" xref="yes"/>
-</segment>
-</net>
-<net name="N$3" class="0">
-<segment>
-<pinref part="U1" gate="G$1" pin="3/PWM"/>
-<wire x1="106.68" y1="33.02" x2="101.6" y2="33.02" width="0.1524" layer="91"/>
 </segment>
 </net>
@@
 <label x="172.72" y="-2.54" size="1.27" layer="95" rot="R180" xref="yes"/>
 </segment>
-</net>
+<segment>
+<pinref part="U1" gate="G$1" pin="2"/>
+<wire x1="106.68" y1="35.56" x2="101.6" y2="35.56" width="0.1524" layer="91"/>
+<label x="101.6" y="35.56" size="1.27" layer="95" rot="R180" xref="yes"/>
+</segment>
+</net>
+<net name="N$1" class="0">
+<segment>
+<pinref part="U1" gate="G$1" pin="11/MOSI"/>
+<wire x1="106.68" y1="12.7" x2="93.98" y2="12.7" width="0.1524" layer="91"/>
+<pinref part="D1" gate="G$1" pin="C"/>
+</segment>
+</net>
+<net name="N$2" class="0">
+<segment>
+<pinref part="LED1" gate="G$1" pin="A"/>
+<pinref part="R1" gate="G$1" pin="2"/>
+</segment>
+</net>
+<net name="N$3" class="0">
+<segment>
+<pinref part="LED2" gate="G$1" pin="A"/>
+<pinref part="R2" gate="G$1" pin="2"/>
+</segment>
+</net>
+<net name="N$4" class="0">
+<segment>
+<pinref part="LED3" gate="G$1" pin="A"/>
+<pinref part="R3" gate="G$1" pin="2"/>
+</segment>
+</net>
+<net name="N$5" class="0">
+<segment>
+<pinref part="LED4" gate="G$1" pin="A"/>
+<pinref part="R4" gate="G$1" pin="2"/>
+</segment>
+</net>
+<net name="N$6" class="0">
+<segment>
+<pinref part="LED5" gate="G$1" pin="A"/>
+<pinref part="R5" gate="G$1" pin="2"/>
+</segment>
+</net>
+<net name="LED-GOOD" class="0">
+<segment>
+<pinref part="R1" gate="G$1" pin="1"/>
+<wire x1="233.68" y1="22.86" x2="228.6" y2="22.86" width="0.1524" layer="91"/>
+<label x="228.6" y="22.86" size="1.27" layer="95" rot="R180" xref="yes"/>
+</segment>
+<segment>
+<pinref part="U1" gate="G$1" pin="7/RX3"/>
+<wire x1="106.68" y1="22.86" x2="101.6" y2="22.86" width="0.1524" layer="91"/>
+<label x="101.6" y="22.86" size="1.27" layer="95" rot="R180" xref="yes"/>
+</segment>
+</net>
+<net name="LED-BAD" class="0">
+<segment>
+<pinref part="R2" gate="G$1" pin="1"/>
+<wire x1="233.68" y1="12.7" x2="228.6" y2="12.7" width="0.1524" layer="91"/>
+<label x="228.6" y="12.7" size="1.27" layer="95" rot="R180" xref="yes"/>
+</segment>
+<segment>
+<pinref part="U1" gate="G$1" pin="6/PWM"/>
+<wire x1="106.68" y1="25.4" x2="101.6" y2="25.4" width="0.1524" layer="91"/>
+<label x="101.6" y="25.4" size="1.27" layer="95" rot="R180" xref="yes"/>
+</segment>
+</net>
+<net name="LED-DATA-UP" class="0">
+<segment>
+<pinref part="R3" gate="G$1" pin="1"/>
+<wire x1="233.68" y1="2.54" x2="228.6" y2="2.54" width="0.1524" layer="91"/>
+<label x="228.6" y="2.54" size="1.27" layer="95" rot="R180" xref="yes"/>
+</segment>
+<segment>
+<pinref part="U1" gate="G$1" pin="5/PWM"/>
+<wire x1="106.68" y1="27.94" x2="101.6" y2="27.94" width="0.1524" layer="91"/>
+<label x="101.6" y="27.94" size="1.27" layer="95" rot="R180" xref="yes"/>
+</segment>
+</net>
+<net name="LED-DATA-DOWN" class="0">
+<segment>
+<pinref part="R4" gate="G$1" pin="1"/>
+<wire x1="233.68" y1="-7.62" x2="228.6" y2="-7.62" width="0.1524" layer="91"/>
+<label x="228.6" y="-7.62" size="1.27" layer="95" rot="R180" xref="yes"/>
+</segment>
+<segment>
+<pinref part="U1" gate="G$1" pin="4/PWM"/>
+<wire x1="106.68" y1="30.48" x2="101.6" y2="30.48" width="0.1524" layer="91"/>
+<label x="101.6" y="30.48" size="1.27" layer="95" rot="R180" xref="yes"/>
+</segment>
+</net>
+<net name="LED-V" class="0">
+<segment>
+<pinref part="R5" gate="G$1" pin="1"/>
+<wire x1="233.68" y1="-17.78" x2="228.6" y2="-17.78" width="0.1524" layer="91"/>
+<label x="228.6" y="-17.78" size="1.27" layer="95" rot="R180" xref="yes"/>
+</segment>
+<segment>
+<pinref part="U1" gate="G$1" pin="3/PWM"/>
+<wire x1="106.68" y1="33.02" x2="101.6" y2="33.02" width="0.1524" layer="91"/>
+<label x="101.6" y="33.02" size="1.27" layer="95" rot="R180" xref="yes"/>
+</segment>
+</net>

Commit message: work on programmer pcb
Parts:
- added C1: (no value), dirtcheaprx:CAP_POLPTH1
- added C2: (no value), dirtcheaprx:CAPPTH2
- added D2: (no value), dirtcheaprx:DIODESOD
- added IC1: (no value), dirtcheaprx:V_REG_LM1117SOT223
- added S3: (no value), dirtcheaprx:TAC_SWITCHPTH
- added X4: ESP01, dirtcheaprx:ESP01
Connections:
- new net N$7: D2.C, U1.12/MISO
- new net RX2: U1.10/TX2/PWM, X4.RXD
- new net SCANNER-RST: U1.8/TX3, X4.RST
- new net TX2: U1.9/RX2/PWM, X4.TXD
- net +3V3: now also C2.1, IC1.OUT, IC1.OUT@1, X4.CH_PD, X4.GPIO0(P), X4.VCC; no longer U1.3.3V
- net BOOT: now also D2.A, S3.1, S3.2; no longer U1.12/MISO
- net GND: now also C1.-, C2.2, IC1.ADJ, S3.3, S3.4, X4.GND
- net VIN: now also C1.+, IC1.IN
Changed lines of the file:
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@@
 <part name="R5" library="dirtcheaprx" deviceset="RESISTOR" device="0603-RES"/>
 <part name="GND7" library="dirtcheaprx" deviceset="GND" device=""/>
+<part name="D2" library="dirtcheaprx" deviceset="DIODE" device="SOD"/>
+<part name="S3" library="dirtcheaprx" deviceset="TAC_SWITCH" device="PTH"/>
+<part name="GND8" library="dirtcheaprx" deviceset="GND" device=""/>
+<part name="X4" library="dirtcheaprx" deviceset="ESP01" device=""/>
+<part name="GND9" library="dirtcheaprx" deviceset="GND" device=""/>
+<part name="IC1" library="dirtcheaprx" deviceset="V_REG_LM1117" device="SOT223"/>
+<part name="GND10" library="dirtcheaprx" deviceset="GND" device=""/>
+<part name="C1" library="dirtcheaprx" deviceset="CAP_POL" device="PTH1"/>
+<part name="C2" library="dirtcheaprx" deviceset="CAP" device="PTH2"/>
 </parts>
 <sheets>
@@
 <instance part="R5" gate="G$1" x="238.76" y="-17.78"/>
 <instance part="GND7" gate="1" x="254" y="-25.4"/>
+<instance part="D2" gate="G$1" x="91.44" y="7.62"/>
+<instance part="S3" gate="S" x="182.88" y="-48.26"/>
+<instance part="GND8" gate="1" x="190.5" y="-55.88"/>
+<instance part="X4" gate="G$1" x="53.34" y="-30.48"/>
+<instance part="GND9" gate="1" x="27.94" y="-17.78"/>
+<instance part="IC1" gate="G$1" x="101.6" y="-58.42"/>
+<instance part="GND10" gate="1" x="86.36" y="-78.74"/>
+<instance part="C1" gate="G$1" x="86.36" y="-66.04"/>
+<instance part="C2" gate="G$1" x="116.84" y="-68.58"/>
 </instances>
 <busses>
@@
 </segment>
 <segment>
-<pinref part="U1" gate="G$1" pin="3.3V"/>
-<wire x1="152.4" y1="38.1" x2="157.48" y2="38.1" width="0.1524" layer="91"/>
-<label x="157.48" y="38.1" size="1.27" layer="95" xref="yes"/>
+<pinref part="X4" gate="G$1" pin="GPIO0(P)"/>
+<wire x1="35.56" y1="-27.94" x2="30.48" y2="-27.94" width="0.1524" layer="91"/>
+<label x="30.48" y="-27.94" size="1.27" layer="95" rot="R180" xref="yes"/>
+</segment>
+<segment>
+<pinref part="X4" gate="G$1" pin="VCC"/>
+<wire x1="68.58" y1="-30.48" x2="83.82" y2="-30.48" width="0.1524" layer="91"/>
+<pinref part="X4" gate="G$1" pin="CH_PD"/>
+<wire x1="83.82" y1="-30.48" x2="91.44" y2="-30.48" width="0.1524" layer="91"/>
+<wire x1="68.58" y1="-25.4" x2="83.82" y2="-25.4" width="0.1524" layer="91"/>
+<wire x1="83.82" y1="-25.4" x2="83.82" y2="-30.48" width="0.1524" layer="91"/>
+<label x="91.44" y="-30.48" size="1.27" layer="95" xref="yes"/>
+</segment>
+<segment>
+<pinref part="IC1" gate="G$1" pin="OUT@1"/>
+<pinref part="C2" gate="G$1" pin="1"/>
+<wire x1="109.22" y1="-60.96" x2="116.84" y2="-60.96" width="0.1524" layer="91"/>
+<wire x1="116.84" y1="-60.96" x2="116.84" y2="-63.5" width="0.1524" layer="91"/>
+<pinref part="IC1" gate="G$1" pin="OUT"/>
+<wire x1="109.22" y1="-58.42" x2="116.84" y2="-58.42" width="0.1524" layer="91"/>
+<wire x1="116.84" y1="-58.42" x2="116.84" y2="-60.96" width="0.1524" layer="91"/>
+<wire x1="116.84" y1="-58.42" x2="121.92" y2="-58.42" width="0.1524" layer="91"/>
+<label x="121.92" y="-58.42" size="1.27" layer="95" xref="yes"/>
+<junction x="116.84" y="-60.96"/>
+<junction x="116.84" y="-58.42"/>
 </segment>
 </net>
@@
 <wire x1="175.26" y1="-27.94" x2="175.26" y2="-25.4" width="0.1524" layer="91"/>
 <label x="170.18" y="-25.4" size="1.27" layer="95" rot="R180" xref="yes"/>
+<junction x="175.26" y="-25.4"/>
 </segment>
 </net>
@@
 </segment>
 <segment>
-<pinref part="U1" gate="G$1" pin="12/MISO"/>
-<wire x1="106.68" y1="10.16" x2="101.6" y2="10.16" width="0.1524" layer="91"/>
-<label x="101.6" y="10.16" size="1.27" layer="95" rot="R180" xref="yes"/>
+<pinref part="D2" gate="G$1" pin="A"/>
+<wire x1="88.9" y1="7.62" x2="83.82" y2="7.62" width="0.1524" layer="91"/>
+<label x="83.82" y="7.62" size="1.27" layer="95" rot="R180" xref="yes"/>
+</segment>
+<segment>
+<pinref part="S3" gate="S" pin="1"/>
+<wire x1="177.8" y1="-48.26" x2="175.26" y2="-48.26" width="0.1524" layer="91"/>
+<pinref part="S3" gate="S" pin="2"/>
+<wire x1="175.26" y1="-48.26" x2="170.18" y2="-48.26" width="0.1524" layer="91"/>
+<wire x1="177.8" y1="-50.8" x2="175.26" y2="-50.8" width="0.1524" layer="91"/>
+<wire x1="175.26" y1="-50.8" x2="175.26" y2="-48.26" width="0.1524" layer="91"/>
+<label x="170.18" y="-48.26" size="1.27" layer="95" rot="R180" xref="yes"/>
+<junction x="175.26" y="-48.26"/>
 </segment>
 </net>
@@
 <wire x1="190.5" y1="-5.08" x2="190.5" y2="-7.62" width="0.1524" layer="91"/>
 <wire x1="187.96" y1="-5.08" x2="190.5" y2="-5.08" width="0.1524" layer="91"/>
+<junction x="190.5" y="-5.08"/>
 </segment>
 <segment>
@@
 <wire x1="190.5" y1="-27.94" x2="190.5" y2="-30.48" width="0.1524" layer="91"/>
 <wire x1="187.96" y1="-27.94" x2="190.5" y2="-27.94" width="0.1524" layer="91"/>
+<junction x="190.5" y="-27.94"/>
 </segment>
 <segment>
@@
 <pinref part="LED2" gate="G$1" pin="C"/>
 <wire x1="251.46" y1="12.7" x2="254" y2="12.7" width="0.1524" layer="91"/>
+<junction x="254" y="12.7"/>
+<junction x="254" y="2.54"/>
+<junction x="254" y="-7.62"/>
+<junction x="254" y="-17.78"/>
+</segment>
+<segment>
+<pinref part="S3" gate="S" pin="3"/>
+<pinref part="GND8" gate="1" pin="GND"/>
+<wire x1="187.96" y1="-48.26" x2="190.5" y2="-48.26" width="0.1524" layer="91"/>
+<wire x1="190.5" y1="-48.26" x2="190.5" y2="-50.8" width="0.1524" layer="91"/>
+<pinref part="S3" gate="S" pin="4"/>
+<wire x1="190.5" y1="-50.8" x2="190.5" y2="-53.34" width="0.1524" layer="91"/>
+<wire x1="187.96" y1="-50.8" x2="190.5" y2="-50.8" width="0.1524" layer="91"/>
+<junction x="190.5" y="-50.8"/>
+</segment>
+<segment>
+<pinref part="X4" gate="G$1" pin="GND"/>
+<wire x1="35.56" y1="-22.86" x2="33.02" y2="-22.86" width="0.1524" layer="91"/>
+<wire x1="33.02" y1="-22.86" x2="33.02" y2="-12.7" width="0.1524" layer="91"/>
+<wire x1="33.02" y1="-12.7" x2="27.94" y2="-12.7" width="0.1524" layer="91"/>
+<pinref part="GND9" gate="1" pin="GND"/>
+<wire x1="27.94" y1="-12.7" x2="27.94" y2="-15.24" width="0.1524" layer="91"/>
+</segment>
+<segment>
+<pinref part="C1" gate="G$1" pin="-"/>
+<pinref part="GND10" gate="1" pin="GND"/>
+<wire x1="86.36" y1="-71.12" x2="86.36" y2="-73.66" width="0.1524" layer="91"/>
+<pinref part="IC1" gate="G$1" pin="ADJ"/>
+<wire x1="86.36" y1="-73.66" x2="86.36" y2="-76.2" width="0.1524" layer="91"/>
+<wire x1="86.36" y1="-73.66" x2="101.6" y2="-73.66" width="0.1524" layer="91"/>
+<wire x1="101.6" y1="-73.66" x2="101.6" y2="-66.04" width="0.1524" layer="91"/>
+<pinref part="C2" gate="G$1" pin="2"/>
+<wire x1="101.6" y1="-73.66" x2="116.84" y2="-73.66" width="0.1524" layer="91"/>
+<wire x1="116.84" y1="-73.66" x2="116.84" y2="-71.12" width="0.1524" layer="91"/>
+<junction x="101.6" y="-73.66"/>
+<junction x="86.36" y="-73.66"/>
 </segment>
 </net>
@@
 <wire x1="152.4" y1="40.64" x2="157.48" y2="40.64" width="0.1524" layer="91"/>
 <label x="157.48" y="40.64" size="1.27" layer="95" xref="yes"/>
+</segment>
+<segment>
+<pinref part="IC1" gate="G$1" pin="IN"/>
+<pinref part="C1" gate="G$1" pin="+"/>
+<wire x1="93.98" y1="-58.42" x2="86.36" y2="-58.42" width="0.1524" layer="91"/>
+<wire x1="86.36" y1="-58.42" x2="86.36" y2="-63.5" width="0.1524" layer="91"/>
+<wire x1="86.36" y1="-58.42" x2="81.28" y2="-58.42" width="0.1524" layer="91"/>
+<label x="81.28" y="-58.42" size="1.27" layer="95" rot="R180" xref="yes"/>
+<junction x="86.36" y="-58.42"/>
 </segment>
 </net>
@@
 <wire x1="175.26" y1="-5.08" x2="175.26" y2="-2.54" width="0.1524" layer="91"/>
 <label x="172.72" y="-2.54" size="1.27" layer="95" rot="R180" xref="yes"/>
+<junction x="175.26" y="-2.54"/>
 </segment>
 <segment>
@@
 </segment>
 </net>
+<net name="N$7" class="0">
+<segment>
+<pinref part="U1" gate="G$1" pin="12/MISO"/>
+<wire x1="106.68" y1="10.16" x2="96.52" y2="10.16" width="0.1524" layer="91"/>
+<wire x1="96.52" y1="10.16" x2="96.52" y2="7.62" width="0.1524" layer="91"/>
+<wire x1="96.52" y1="7.62" x2="93.98" y2="7.62" width="0.1524" layer="91"/>
+<pinref part="D2" gate="G$1" pin="C"/>
+</segment>
+</net>
+<net name="TX2" class="0">
+<segment>
+<pinref part="U1" gate="G$1" pin="9/RX2/PWM"/>
+<wire x1="106.68" y1="17.78" x2="104.14" y2="17.78" width="0.1524" layer="91"/>
+<label x="104.14" y="17.78" size="1.27" layer="95" rot="R180" xref="yes"/>
+</segment>
+<segment>
+<pinref part="X4" gate="G$1" pin="TXD"/>
+<wire x1="68.58" y1="-22.86" x2="73.66" y2="-22.86" width="0.1524" layer="91"/>
+<label x="73.66" y="-22.86" size="1.27" layer="95" xref="yes"/>
+</segment>
+</net>
+<net name="RX2" class="0">
+<segment>
+<pinref part="U1" gate="G$1" pin="10/TX2/PWM"/>
+<wire x1="106.68" y1="15.24" x2="104.14" y2="15.24" width="0.1524" layer="91"/>
+<label x="104.14" y="15.24" size="1.27" layer="95" rot="R180" xref="yes"/>
+</segment>
+<segment>
+<pinref part="X4" gate="G$1" pin="RXD"/>
+<wire x1="35.56" y1="-30.48" x2="30.48" y2="-30.48" width="0.1524" layer="91"/>
+<label x="30.48" y="-30.48" size="1.27" layer="95" rot="R180" xref="yes"/>
+</segment>
+</net>
+<net name="SCANNER-RST" class="0">
+<segment>
+<pinref part="X4" gate="G$1" pin="RST"/>
+<wire x1="68.58" y1="-27.94" x2="71.12" y2="-27.94" width="0.1524" layer="91"/>
+<label x="71.12" y="-27.94" size="1.27" layer="95" xref="yes"/>
+</segment>
+<segment>
+<pinref part="U1" gate="G$1" pin="8/TX3"/>
+<wire x1="106.68" y1="20.32" x2="101.6" y2="20.32" width="0.1524" layer="91"/>
+<label x="101.6" y="20.32" size="1.27" layer="95" rot="R180" xref="yes"/>
+</segment>
+</net>
